File: pcb/macrocat.kicad_sch (KiCad schematic)
At the start: 52 parts, among them J1 USB-C Connector, U1 ATmega32U4-M, Y1 16M

Commit message: create 3d model
Parts:
- KNOB1: footprint Rotary_Encoder:RotaryEncoder_Alps_EC11E-Switch_Vertical_H20mm -> macrocat:RotaryEncoder_Alps_EC11E-Switch_Vertical_H20mm
- MX1, MX10, MX11, MX12, MX13, MX14, MX15, MX16, MX2, MX3, MX4, MX5, MX6, MX7, MX8, MX9: footprint MX_Only:MXOnly-1U-Hotswap -> macrocat:MXOnly-1U-Hotswap
Changed lines of the file:
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@@
       (effects (font (size 0.508 0.508)))
     )
-    (property "Footprint" "MX_Only:MXOnly-1U-Hotswap" (id 2) (at 175.895 70.485 0)
+    (property "Footprint" "macrocat:MXOnly-1U-Hotswap" (id 2) (at 175.895 70.485 0)
       (effects (font (size 1.524 1.524)) hide)
     )
@@
       (effects (font (size 0.508 0.508)))
     )
-    (property "Footprint" "MX_Only:MXOnly-1U-Hotswap" (id 2) (at 203.835 92.075 0)
+    (property "Footprint" "macrocat:MXOnly-1U-Hotswap" (id 2) (at 203.835 92.075 0)
       (effects (font (size 1.524 1.524)) hide)
     )
@@
       (effects (font (size 0.508 0.508)))
     )
-    (property "Footprint" "MX_Only:MXOnly-1U-Hotswap" (id 2) (at 175.895 92.075 0)
+    (property "Footprint" "macrocat:MXOnly-1U-Hotswap" (id 2) (at 175.895 92.075 0)
       (effects (font (size 1.524 1.524)) hide)
     )
@@
       (effects (font (size 0.508 0.508)))
     )
-    (property "Footprint" "MX_Only:MXOnly-1U-Hotswap" (id 2) (at 203.835 113.665 0)
+    (property "Footprint" "macrocat:MXOnly-1U-Hotswap" (id 2) (at 203.835 113.665 0)
       (effects (font (size 1.524 1.524)) hide)
     )
@@
       (effects (font (size 0.508 0.508)))
     )
-    (property "Footprint" "MX_Only:MXOnly-1U-Hotswap" (id 2) (at 160.655 92.075 0)
+    (property "Footprint" "macrocat:MXOnly-1U-Hotswap" (id 2) (at 160.655 92.075 0)
       (effects (font (size 1.524 1.524)) hide)
     )
@@
       (effects (font (size 0.508 0.508)))
     )
-    (property "Footprint" "MX_Only:MXOnly-1U-Hotswap" (id 2) (at 175.895 135.255 0)
+    (property "Footprint" "macrocat:MXOnly-1U-Hotswap" (id 2) (at 175.895 135.255 0)
       (effects (font (size 1.524 1.524)) hide)
     )
@@
       (effects (font (size 0.508 0.508)))
     )
-    (property "Footprint" "MX_Only:MXOnly-1U-Hotswap" (id 2) (at 175.895 113.665 0)
+    (property "Footprint" "macrocat:MXOnly-1U-Hotswap" (id 2) (at 175.895 113.665 0)
       (effects (font (size 1.524 1.524)) hide)
     )
@@
       (effects (font (size 0.508 0.508)))
     )
-    (property "Footprint" "MX_Only:MXOnly-1U-Hotswap" (id 2) (at 189.865 135.255 0)
+    (property "Footprint" "macrocat:MXOnly-1U-Hotswap" (id 2) (at 189.865 135.255 0)
       (effects (font (size 1.524 1.524)) hide)
     )
@@
       (effects (font (size 0.508 0.508)))
     )
-    (property "Footprint" "MX_Only:MXOnly-1U-Hotswap" (id 2) (at 160.655 135.255 0)
+    (property "Footprint" "macrocat:MXOnly-1U-Hotswap" (id 2) (at 160.655 135.255 0)
       (effects (font (size 1.524 1.524)) hide)
     )
@@
       (effects (font (size 0.508 0.508)))
     )
-    (property "Footprint" "MX_Only:MXOnly-1U-Hotswap" (id 2) (at 160.655 70.485 0)
+    (property "Footprint" "macrocat:MXOnly-1U-Hotswap" (id 2) (at 160.655 70.485 0)
       (effects (font (size 1.524 1.524)) hide)
     )
@@
       (effects (font (size 0.508 0.508)))
     )
-    (property "Footprint" "MX_Only:MXOnly-1U-Hotswap" (id 2) (at 203.835 70.485 0)
+    (property "Footprint" "macrocat:MXOnly-1U-Hotswap" (id 2) (at 203.835 70.485 0)
       (effects (font (size 1.524 1.524)) hide)
     )
@@
       (effects (font (size 0.508 0.508)))
     )
-    (property "Footprint" "MX_Only:MXOnly-1U-Hotswap" (id 2) (at 189.865 92.075 0)
+    (property "Footprint" "macrocat:MXOnly-1U-Hotswap" (id 2) (at 189.865 92.075 0)
       (effects (font (size 1.524 1.524)) hide)
     )
@@
     (property "Reference" "KNOB1" (id 0) (at 124.46 90.17 0))
     (property "Value" "RotaryEncoder_Switch" (id 1) (at 124.46 92.71 0))
-    (property "Footprint" "Rotary_Encoder:RotaryEncoder_Alps_EC11E-Switch_Vertical_H20mm" (id 2) (at 120.65 96.266 0)
+    (property "Footprint" "macrocat:RotaryEncoder_Alps_EC11E-Switch_Vertical_H20mm" (id 2) (at 120.65 96.266 0)
       (effects (font (size 1.27 1.27)) hide)
     )
@@
       (effects (font (size 0.508 0.508)))
     )
-    (property "Footprint" "MX_Only:MXOnly-1U-Hotswap" (id 2) (at 189.865 70.485 0)
+    (property "Footprint" "macrocat:MXOnly-1U-Hotswap" (id 2) (at 189.865 70.485 0)
       (effects (font (size 1.524 1.524)) hide)
     )
@@
       (effects (font (size 0.508 0.508)))
     )
-    (property "Footprint" "MX_Only:MXOnly-1U-Hotswap" (id 2) (at 160.655 113.665 0)
+    (property "Footprint" "macrocat:MXOnly-1U-Hotswap" (id 2) (at 160.655 113.665 0)
       (effects (font (size 1.524 1.524)) hide)
     )
@@
       (effects (font (size 0.508 0.508)))
     )
-    (property "Footprint" "MX_Only:MXOnly-1U-Hotswap" (id 2) (at 203.835 135.255 0)
+    (property "Footprint" "macrocat:MXOnly-1U-Hotswap" (id 2) (at 203.835 135.255 0)
       (effects (font (size 1.524 1.524)) hide)
     )
@@
       (effects (font (size 0.508 0.508)))
     )
-    (property "Footprint" "MX_Only:MXOnly-1U-Hotswap" (id 2) (at 189.865 113.665 0)
+    (property "Footprint" "macrocat:MXOnly-1U-Hotswap" (id 2) (at 189.865 113.665 0)
       (effects (font (size 1.524 1.524)) hide)
     )
@@
     )
     (path "/7ce1fa23-e6c8-4f4d-a700-97b0bc833646"
-      (reference "KNOB1") (unit 1) (value "RotaryEncoder_Switch") (footprint "Rotary_Encoder:RotaryEncoder_Alps_EC11E-Switch_Vertical_H20mm")
+      (reference "KNOB1") (unit 1) (value "RotaryEncoder_Switch") (footprint "macrocat:RotaryEncoder_Alps_EC11E-Switch_Vertical_H20mm")
     )
     (path "/4dc965b4-2750-4e34-ac33-80b79bca93bb"
-      (reference "MX1") (unit 1) (value "MX-NoLED") (footprint "MX_Only:MXOnly-1U-Hotswap")
+      (reference "MX1") (unit 1) (value "MX-NoLED") (footprint "macrocat:MXOnly-1U-Hotswap")
     )
     (path "/22960c85-9995-45f2-b052-dec16cd9fb31"
-      (reference "MX2") (unit 1) (value "MX-NoLED") (footprint "MX_Only:MXOnly-1U-Hotswap")
+      (reference "MX2") (unit 1) (value "MX-NoLED") (footprint "macrocat:MXOnly-1U-Hotswap")
     )
     (path "/bf126b27-eb87-493e-8d25-04bcb3a7a9a7"
-      (reference "MX3") (unit 1) (value "MX-NoLED") (footprint "MX_Only:MXOnly-1U-Hotswap")
+      (reference "MX3") (unit 1) (value "MX-NoLED") (footprint "macrocat:MXOnly-1U-Hotswap")
     )
     (path "/495c00a9-57e8-4082-8fd8-85e656975b00"
-      (reference "MX4") (unit 1) (value "MX-NoLED") (footprint "MX_Only:MXOnly-1U-Hotswap")
+      (reference "MX4") (unit 1) (value "MX-NoLED") (footprint "macrocat:MXOnly-1U-Hotswap")
     )
     (path "/00116c46-2b19-4ef8-a8d5-827de780bce9"
-      (reference "MX5") (unit 1) (value "MX-NoLED") (footprint "MX_Only:MXOnly-1U-Hotswap")
+      (reference "MX5") (unit 1) (value "MX-NoLED") (footprint "macrocat:MXOnly-1U-Hotswap")
     )
     (path "/02db5ce1-8dd7-4779-9959-08d807e3fdb2"
-      (reference "MX6") (unit 1) (value "MX-NoLED") (footprint "MX_Only:MXOnly-1U-Hotswap")
+      (reference "MX6") (unit 1) (value "MX-NoLED") (footprint "macrocat:MXOnly-1U-Hotswap")
     )
     (path "/30463a3a-46f9-4746-a929-c7807f5ef36b"
-      (reference "MX7") (unit 1) (value "MX-NoLED") (footprint "MX_Only:MXOnly-1U-Hotswap")
+      (reference "MX7") (unit 1) (value "MX-NoLED") (footprint "macrocat:MXOnly-1U-Hotswap")
     )
     (path "/302d4c94-1f0a-48e8-818d-2faf4246daef"
-      (reference "MX8") (unit 1) (value "MX-NoLED") (footprint "MX_Only:MXOnly-1U-Hotswap")
+      (reference "MX8") (unit 1) (value "MX-NoLED") (footprint "macrocat:MXOnly-1U-Hotswap")
     )
     (path "/8a0f3145-9e31-47f7-addf-c6575c773c53"
-      (reference "MX9") (unit 1) (value "MX-NoLED") (footprint "MX_Only:MXOnly-1U-Hotswap")
+      (reference "MX9") (unit 1) (value "MX-NoLED") (footprint "macrocat:MXOnly-1U-Hotswap")
     )
     (path "/63425f6a-695c-4807-9f43-7fec9922a465"
-      (reference "MX10") (unit 1) (value "MX-NoLED") (footprint "MX_Only:MXOnly-1U-Hotswap")
+      (reference "MX10") (unit 1) (value "MX-NoLED") (footprint "macrocat:MXOnly-1U-Hotswap")
     )
     (path "/f99943a0-11ef-43bb-8f57-ee98ff71d17b"
-      (reference "MX11") (unit 1) (value "MX-NoLED") (footprint "MX_Only:MXOnly-1U-Hotswap")
+      (reference "MX11") (unit 1) (value "MX-NoLED") (footprint "macrocat:MXOnly-1U-Hotswap")
     )
     (path "/4815b4bc-933e-4212-adad-d9dccf508edc"
-      (reference "MX12") (unit 1) (value "MX-NoLED") (footprint "MX_Only:MXOnly-1U-Hotswap")
+      (reference "MX12") (unit 1) (value "MX-NoLED") (footprint "macrocat:MXOnly-1U-Hotswap")
     )
     (path "/5923c8bf-cda5-477c-ad14-b2f3f65081b2"
-      (reference "MX13") (unit 1) (value "MX-NoLED") (footprint "MX_Only:MXOnly-1U-Hotswap")
+      (reference "MX13") (unit 1) (value "MX-NoLED") (footprint "macrocat:MXOnly-1U-Hotswap")
     )
     (path "/023d540f-6655-4df7-a0f4-2a77e896da1b"
-      (reference "MX14") (unit 1) (value "MX-NoLED") (footprint "MX_Only:MXOnly-1U-Hotswap")
+      (reference "MX14") (unit 1) (value "MX-NoLED") (footprint "macrocat:MXOnly-1U-Hotswap")
     )
     (path "/14d337e6-ff30-40ce-9856-840e5b5ed652"
-      (reference "MX15") (unit 1) (value "MX-NoLED") (footprint "MX_Only:MXOnly-1U-Hotswap")
+      (reference "MX15") (unit 1) (value "MX-NoLED") (footprint "macrocat:MXOnly-1U-Hotswap")
     )
     (path "/c35b87b8-f2aa-46a3-860a-44917266d4b3"
-      (reference "MX16") (unit 1) (value "MX-NoLED") (footprint "MX_Only:MXOnly-1U-Hotswap")
+      (reference "MX16") (unit 1) (value "MX-NoLED") (footprint "macrocat:MXOnly-1U-Hotswap")
     )
     (path "/c79ca30d-bb72-469e-a0b1-dceb03b0389c"
